Commit message: Fixed URDF

File: StaubliURDF/arm_2/robots/arm_2.urdf (robot description, URDF)
Before this commit: robot Arm_2, 7 links, 6 joints
Links:
- link Link_1: geometry collision mesh filename=package://arm_2/meshes/Link_1.STL; visual mesh filename=package://arm_2/meshes/Link_1.STL
- link Link_2: geometry collision mesh filename=package://arm_2/meshes/Link_2.STL; visual mesh filename=package://arm_2/meshes/Link_2.STL
- link Link_3: geometry collision mesh filename=package://arm_2/meshes/Link_3.STL; visual mesh filename=package://arm_2/meshes/Link_3.STL
- link Link_4: geometry collision mesh filename=package://arm_2/meshes/Link_4.STL; visual mesh filename=package://arm_2/meshes/Link_4.STL
- link Link_5: geometry collision mesh filename=package://arm_2/meshes/Link_5.STL; visual mesh filename=package://arm_2/meshes/Link_5.STL
- link Link_6: geometry collision mesh filename=package://arm_2/meshes/Link_6.STL; visual mesh filename=package://arm_2/meshes/Link_6.STL
- link base_link: geometry collision mesh filename=package://arm_2/meshes/base_link.STL; visual mesh filename=package://arm_2/meshes/base_link.STL
Joints:
- joint Joint_1: origin xyz=0 0 0.21 rpy=-6.123E-17 0 0 -> xyz=0 0 0.21 rpy=0 0 0
